File: hw/ehx_dmm_clk.sch (KiCad schematic (older format))
At the start: 35 parts, among them J1 Conn_01x06, J2 Conn_01x02, J3 Conn_01x02, J4 Conn_01x03, J5 Conn_01x02, J6 Conn_01x02, Q1 2N5401, Q2 2N5401, U1 PIC16F18326-P, U2 LM7905_TO220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

Commit message: Added some mounting holes
Parts:
- added H1, H2, H3, H4: MountingHole, MountingHole:MountingHole_3mm, symbol Mechanical:MountingHole
Changed lines of the file:
@@
 Wire Wire Line
 	4800 3450 4800 3850
+$Comp
+L Mechanical:MountingHole H2
+U 1 1 5F45102C
+P 4400 7300
+F 0 "H2" H 4500 7346 50  0000 L CNN
+F 1 "MountingHole" H 4500 7255 50  0000 L CNN
+F 2 "MountingHole:MountingHole_3mm" H 4400 7300 50  0001 C CNN
+F 3 "~" H 4400 7300 50  0001 C CNN
+	1    4400 7300
+	1    0    0    -1
+$EndComp
+$Comp
+L Mechanical:MountingHole H4
+U 1 1 5F451148
+P 5350 7300
+F 0 "H4" H 5450 7346 50  0000 L CNN
+F 1 "MountingHole" H 5450 7255 50  0000 L CNN
+F 2 "MountingHole:MountingHole_3mm" H 5350 7300 50  0001 C CNN
+F 3 "~" H 5350 7300 50  0001 C CNN
+	1    5350 7300
+	1    0    0    -1
+$EndComp
+$Comp
+L Mechanical:MountingHole H1
+U 1 1 5F451201
+P 4400 7000
+F 0 "H1" H 4500 7046 50  0000 L CNN
+F 1 "MountingHole" H 4500 6955 50  0000 L CNN
+F 2 "MountingHole:MountingHole_3mm" H 4400 7000 50  0001 C CNN
+F 3 "~" H 4400 7000 50  0001 C CNN
+	1    4400 7000
+	1    0    0    -1
+$EndComp
+$Comp
+L Mechanical:MountingHole H3
+U 1 1 5F4512BF
+P 5350 7000
+F 0 "H3" H 5450 7046 50  0000 L CNN
+F 1 "MountingHole" H 5450 6955 50  0000 L CNN
+F 2 "MountingHole:MountingHole_3mm" H 5350 7000 50  0001 C CNN
+F 3 "~" H 5350 7000 50  0001 C CNN
+	1    5350 7000
+	1    0    0    -1
+$EndComp
 $EndSCHEMATC

Commit message: Huge commit. Major changes to board size, layout, footprints, etc. All to get the design to fit into the enclosure
Parts:
- C1, C4: footprint Capacitor_THT:CP_Radial_D12.5mm_P5.00mm -> Capacitor_THT:CP_Radial_D8.0mm_P2.50mm
- R1, R10, R11, R12, R13, R14, R2, R5, R6, R9: footprint Resistor_THT:R_Axial_DIN0207_L6.3mm_D2.5mm_P7.62mm_Horizontal -> Resistor_THT:R_Axial_DIN0207_L6.3mm_D2.5mm_P2.54mm_Vertical
Changed lines of the file:
@@
 F 0 "R9" V 6245 3650 50  0000 C CNN
 F 1 "1K" V 6336 3650 50  0000 C CNN
-F 2 "Resistor_THT:R_Axial_DIN0207_L6.3mm_D2.5mm_P7.62mm_Horizontal" V 6490 3640 50  0001 C CNN
+F 2 "Resistor_THT:R_Axial_DIN0207_L6.3mm_D2.5mm_P2.54mm_Vertical" V 6490 3640 50  0001 C CNN
 F 3 "" H 6450 3650 50  0001 C CNN
 	1    6450 3650
@@
 F 0 "R11" H 7068 4346 50  0000 L CNN
 F 1 "4.7k" H 7068 4255 50  0000 L CNN
-F 2 "Resistor_THT:R_Axial_DIN0207_L6.3mm_D2.5mm_P7.62mm_Horizontal" V 7040 4290 50  0001 C CNN
+F 2 "Resistor_THT:R_Axial_DIN0207_L6.3mm_D2.5mm_P2.54mm_Vertical" V 7040 4290 50  0001 C CNN
 F 3 "" H 7000 4300 50  0001 C CNN
 	1    7000 4300
@@
 F 0 "C1" H 1615 6646 50  0000 L CNN
 F 1 "33uF" H 1615 6555 50  0000 L CNN
-F 2 "Capacitor_THT:CP_Radial_D12.5mm_P5.00mm" H 1500 6600 50  0001 C CNN
+F 2 "Capacitor_THT:CP_Radial_D8.0mm_P2.50mm" H 1500 6600 50  0001 C CNN
 F 3 "" H 1500 6600 50  0001 C CNN
 	1    1500 6600
@@
 F 0 "C4" H 3115 6646 50  0000 L CNN
 F 1 "33uF" H 3115 6555 50  0000 L CNN
-F 2 "Capacitor_THT:CP_Radial_D12.5mm_P5.00mm" H 3000 6600 50  0001 C CNN
+F 2 "Capacitor_THT:CP_Radial_D8.0mm_P2.50mm" H 3000 6600 50  0001 C CNN
 F 3 "" H 3000 6600 50  0001 C CNN
 	1    3000 6600
@@
 F 0 "R10" V 6295 5300 50  0000 C CNN
 F 1 "1K" V 6386 5300 50  0000 C CNN
-F 2 "Resistor_THT:R_Axial_DIN0207_L6.3mm_D2.5mm_P7.62mm_Horizontal" V 6540 5290 50  0001 C CNN
+F 2 "Resistor_THT:R_Axial_DIN0207_L6.3mm_D2.5mm_P2.54mm_Vertical" V 6540 5290 50  0001 C CNN
 F 3 "" H 6500 5300 50  0001 C CNN
 	1    6500 5300
@@
 F 0 "R12" H 7068 5996 50  0000 L CNN
 F 1 "4.7k" H 7068 5905 50  0000 L CNN
-F 2 "Resistor_THT:R_Axial_DIN0207_L6.3mm_D2.5mm_P7.62mm_Horizontal" V 7040 5940 50  0001 C CNN
+F 2 "Resistor_THT:R_Axial_DIN0207_L6.3mm_D2.5mm_P2.54mm_Vertical" V 7040 5940 50  0001 C CNN
 F 3 "" H 7000 5950 50  0001 C CNN
 	1    7000 5950
@@
 F 0 "R1" H 1868 2996 50  0000 L CNN
 F 1 "10k" H 1868 2905 50  0000 L CNN
-F 2 "Resistor_THT:R_Axial_DIN0207_L6.3mm_D2.5mm_P7.62mm_Horizontal" V 1840 2940 50  0001 C CNN
+F 2 "Resistor_THT:R_Axial_DIN0207_L6.3mm_D2.5mm_P2.54mm_Vertical" V 1840 2940 50  0001 C CNN
 F 3 "" H 1800 2950 50  0001 C CNN
 	1    1800 2950
@@
 F 0 "R14" H 9568 1096 50  0000 L CNN
 F 1 "47k" H 9568 1005 50  0000 L CNN
-F 2 "Resistor_THT:R_Axial_DIN0207_L6.3mm_D2.5mm_P7.62mm_Horizontal" V 9540 1040 50  0001 C CNN
+F 2 "Resistor_THT:R_Axial_DIN0207_L6.3mm_D2.5mm_P2.54mm_Vertical" V 9540 1040 50  0001 C CNN
 F 3 "" H 9500 1050 50  0001 C CNN
 	1    9500 1050
@@
 F 0 "R13" H 7868 1796 50  0000 L CNN
 F 1 "4.7k" H 7868 1705 50  0000 L CNN
-F 2 "Resistor_THT:R_Axial_DIN0207_L6.3mm_D2.5mm_P7.62mm_Horizontal" V 7840 1740 50  0001 C CNN
+F 2 "Resistor_THT:R_Axial_DIN0207_L6.3mm_D2.5mm_P2.54mm_Vertical" V 7840 1740 50  0001 C CNN
 F 3 "" H 7800 1750 50  0001 C CNN
 	1    7800 1750
@@
 F 0 "R2" H 1868 4746 50  0000 L CNN
 F 1 "10k" H 1868 4655 50  0000 L CNN
-F 2 "Resistor_THT:R_Axial_DIN0207_L6.3mm_D2.5mm_P7.62mm_Horizontal" V 1840 4690 50  0001 C CNN
+F 2 "Resistor_THT:R_Axial_DIN0207_L6.3mm_D2.5mm_P2.54mm_Vertical" V 1840 4690 50  0001 C CNN
 F 3 "" H 1800 4700 50  0001 C CNN
 	1    1800 4700
@@
 F 0 "R5" H 3618 4746 50  0000 L CNN
 F 1 "10k" H 3618 4655 50  0000 L CNN
-F 2 "Resistor_THT:R_Axial_DIN0207_L6.3mm_D2.5mm_P7.62mm_Horizontal" V 3590 4690 50  0001 C CNN
+F 2 "Resistor_THT:R_Axial_DIN0207_L6.3mm_D2.5mm_P2.54mm_Vertical" V 3590 4690 50  0001 C CNN
 F 3 "" H 3550 4700 50  0001 C CNN
 	1    3550 4700
@@
 F 0 "R6" H 4368 5346 50  0000 L CNN
 F 1 "10k" H 4368 5255 50  0000 L CNN
-F 2 "Resistor_THT:R_Axial_DIN0207_L6.3mm_D2.5mm_P7.62mm_Horizontal" V 4340 5290 50  0001 C CNN
+F 2 "Resistor_THT:R_Axial_DIN0207_L6.3mm_D2.5mm_P2.54mm_Vertical" V 4340 5290 50  0001 C CNN
 F 3 "" H 4300 5300 50  0001 C CNN
 	1    4300 5300
